File: KiCad/dyad.kicad_sch (KiCad schematic)
At the start: 0 parts

Commit message: main
Parts:
- added C1, C13, C14, C15, C23, C24, C26, C27, C32: 10uF, Capacitor_SMD:C_0603_1608Metric_Pad1.08x0.95mm_HandSolder, symbol Device:C
- added C10, C11, C12, C19, C3, C4, C6, C7, C8, C9: 100nF, Capacitor_SMD:C_0603_1608Metric_Pad1.08x0.95mm_HandSolder, symbol Device:C
- added C16, C2, C22, C29, C5: 1uF, Capacitor_SMD:C_0603_1608Metric_Pad1.08x0.95mm_HandSolder, symbol Device:C
- added C17, C18: 4.7uF, Capacitor_SMD:C_0603_1608Metric_Pad1.08x0.95mm_HandSolder, symbol Device:C
- added C20, C21: 12pF, Capacitor_SMD:C_0603_1608Metric_Pad1.08x0.95mm_HandSolder, symbol Device:C
- added C25, C28, C30, C31: 0.1uF, Capacitor_SMD:C_0603_1608Metric_Pad1.08x0.95mm_HandSolder, symbol Device:C
- added D1, D6: SS14, Diode_SMD:D_SMA, symbol Diode:SS14
- added D2: MBR340, Diode_THT:D_DO-201AD_P15.24mm_Horizontal, symbol Diode:MBR340
- added D3, D4, D5, D7: LED, LED_SMD:LED_0603_1608Metric_Pad1.05x0.95mm_HandSolder, symbol Device:LED
- added D8: WS2812B-2020, LED_SMD:LED_WS2812B-2020_PLCC4_2.0x2.0mm, symbol LED:WS2812B-2020
- added F1, F2: MF-MSMF110, Fuse:Fuse_1206_3216Metric_Pad1.42x1.75mm_HandSolder, symbol Device:Polyfuse
- added H1, H2, H3, H4: MountingHole_Pad, MountingHole:MountingHole_2.7mm_M2.5_DIN965_Pad, symbol Mechanical:MountingHole_Pad
- added J1: RP2040 USB C, PCM_marbastlib-various:USB_C_Receptacle_HRO_TYPE-C-31-M-12, symbol Connector:USB_C_Receptacle_USB2.0_16P
- added J2: ESP32 USB C, PCM_marbastlib-various:USB_C_Receptacle_HRO_TYPE-C-31-M-12, symbol Connector:USB_C_Receptacle_USB2.0_16P
- added J3: Micro_SD_Card, Connector_Card:microSD_HC_Hirose_DM3AT-SF-PEJM5, symbol Connector:Micro_SD_Card
- added J4: Conn_01x02, Connector_JST:JST_PH_B2B-PH-K_1x02_P2.00mm_Vertical, symbol Connector_Generic:Conn_01x02
- added J5, J7: Conn_01x03, Connector_JST:JST_PH_B3B-PH-K_1x03_P2.00mm_Vertical, symbol Connector_Generic:Conn_01x03
- added J6: Conn_02x20_Counter_Clockwise, Connector_PinHeader_2.54mm:PinHeader_2x20_P2.54mm_Vertical, symbol Connector_Generic:Conn_02x20_Counter_Clockwise
- added J8: Conn_01x04, Connector_JST:JST_PH_B4B-PH-K_1x04_P2.00mm_Vertical, symbol Connector_Generic:Conn_01x04
- added Q1: DMG3414U, Package_TO_SOT_SMD:SOT-23, symbol Transistor_FET:DMG3414U
- added Q2, Q3: Q_NPN_BEC, Package_TO_SOT_SMD:SOT-23, symbol Transistor_BJT:Q_NPN_BEC
- added R1, R2, R3, R4: 5.1k, Resistor_SMD:R_0603_1608Metric_Pad0.98x0.95mm_HandSolder, symbol Device:R
- added R10, R9: 100k, Resistor_SMD:R_0603_1608Metric_Pad0.98x0.95mm_HandSolder, symbol Device:R
- added R11, R12, R13: 4.7k, Resistor_SMD:R_0603_1608Metric_Pad0.98x0.95mm_HandSolder, symbol Device:R
- added R14, R16, R17, R18, R19, R22: 1k, Resistor_SMD:R_0603_1608Metric_Pad0.98x0.95mm_HandSolder, symbol Device:R
- added R15: 0, Resistor_SMD:R_0603_1608Metric_Pad0.98x0.95mm_HandSolder, symbol Device:R
- added R20, R21, R23, R24, R5, R6: 10k, Resistor_SMD:R_0603_1608Metric_Pad0.98x0.95mm_HandSolder, symbol Device:R
- added R7, R8: 27, Resistor_SMD:R_0603_1608Metric_Pad0.98x0.95mm_HandSolder, symbol Device:R
- added SW1: BOOT, Button_Switch_SMD:SW_SPST_B3U-1000P, symbol Switch:SW_Push
- added SW2: EN, Button_Switch_SMD:SW_SPST_B3U-1000P, symbol Switch:SW_Push
- added SW3: GPIO0, Button_Switch_SMD:SW_SPST_B3U-1000P, symbol Switch:SW_Push
- added U1: RP2040, Package_DFN_QFN:QFN-56-1EP_7x7mm_P0.4mm_EP3.2x3.2mm, symbol MCU_RaspberryPi:RP2040
- added U2: AP2112K-3.3, Package_TO_SOT_SMD:SOT-23-5, symbol Regulator_Linear:AP2112K-3.3
- added U3: MCP73831-2-OT, Package_TO_SOT_SMD:SOT-23-5, symbol Battery_Management:MCP73831-2-OT
- added U4: W25Q128JVS, Package_SO:SOIC-8_5.3x5.3mm_P1.27mm, symbol Memory_Flash:W25Q128JVS
- added U5: CP2104, Package_DFN_QFN:QFN-24-1EP_4x4mm_P0.5mm_EP2.6x2.6mm, symbol Interface_USB:CP2104
- added U6: ESP32-WROOM-32E, RF_Module:ESP32-WROOM-32E, symbol RF_Module:ESP32-WROOM-32E
- added Y1: Crystal_GND2, Crystal:Crystal_SMD_3225-4Pin_3.2x2.5mm_HandSoldering, symbol Device:Crystal_GND2
Connections:
- new net: Q2.2 (E), Q3.1 (B), R24.1
- new net: Q2.1 (B), Q3.2 (E), R23.2
- new net: D8.1 (DOUT), J5.2 (Pin_2)
- new net: D3.1 (K), R13.1, U3.1 (STAT)
- new net: D4.2 (A), R13.2
- new net: D1.2 (A), F1.1
- new net: J2.A5 (CC1), R3.1
- new net: J2.B5 (CC2), R4.1
- new net: R7.2, U1.46 (USB_DM)
- new net: J1.A5 (CC1), R1.1
- new net: D6.2 (A), F2.1, F2.2
- new net: D7.2 (A), R22.2
- new net: R10.2, U2.3 (EN)
- new net: D3.2 (A), R11.2
- new net: D5.2 (A), R14.2
- new net: R17.1, Y1.3
- new net: J1.B5 (CC2), R2.1
- new net: R8.1, U1.47 (USB_DP)
- new net: R12.2, U3.5 (PROG)
- new net +1V1: C2.1, C3.1, C4.1, U1.23 (DVDD), U1.45 (VREG_VOUT), U1.50 (DVDD)
- new net +3V3: C1.1, C10.2, C11.2, C12.2, C14.1, C15.1, C16.1, C19.1, C23.1, C24.1, C25.1, C27.1, C28.1, C32.1, C5.2, C6.2, C7.2, C8.2, C9.2, J3.4 (VDD), R15.1, R18.1, R19.1, R20.1, R21.1, R5.2, R6.2, U1.1 (IOVDD), U1.10 (IOVDD), U1.22 (IOVDD), U1.33 (IOVDD), U1.42 (IOVDD), U1.43 (ADC_AVDD), U1.44 (VREG_VIN), U1.48 (USB_VDD), U1.49 (IOVDD), U2.5 (VOUT), U4.8 (VCC), U5.5 (VIO), U5.6 (VDD), U5.7 (REGIN), U6.2 (VDD)
- new net +5V: C13.1, C31.1, D2.1 (K), D8.4 (VDD), J5.1 (Pin_1), Q1.2 (S), R10.1, U2.1 (VIN)
- new net DTR: R24.2, U5.23 (~{DTR})
- new net DUAL_VBUS: C17.1, D1.1 (K), D2.2 (A), D6.1 (K), Q1.1 (G), R11.1, R9.1, U3.4 (V_{DD}), U5.8 (VBUS)
- new net ESP32_EN: C26.2, C29.1, Q2.3 (C), R20.2, SW2.2, U6.3 (EN)
- new net ESPIO_0: C30.1, Q3.3 (C), R21.2, SW3.2, U6.25 (IO0)
- new net ESPIO_12: J6.29 (Pin_29), U6.14 (IO12)
- new net ESPIO_13: J6.30 (Pin_30), U6.16 (IO13)
- new net ESPIO_14: J6.31 (Pin_31), U6.13 (IO14)
- new net ESPIO_15: J6.32 (Pin_32), U6.23 (IO15)
- new net ESPIO_16: U1.11 (GPIO8), U6.27 (IO16)
- new net ESPIO_17: U1.12 (GPIO9), U6.28 (IO17)
- new net ESPIO_18: R22.1, U6.30 (IO18)
- new net ESPIO_19: D8.3 (DIN), U6.31 (IO19)
- new net ESPIO_2: U6.24 (IO2)
- new net ESPIO_21: J8.2 (Pin_2), R18.2, R19.2, U1.13 (GPIO10), U6.33 (IO21)
- new net ESPIO_22: J8.1 (Pin_1), U1.14 (GPIO11), U6.36 (IO22)
- new net ESPIO_23: J6.33 (Pin_33), U6.37 (IO23)
- new net ESPIO_25: J6.34 (Pin_34), U6.10 (IO25)
- new net ESPIO_26: J6.35 (Pin_35), U6.11 (IO26)
- new net ESPIO_27: J6.36 (Pin_36), U6.12 (IO27)
- new net ESPIO_32: J6.37 (Pin_37), U6.8 (IO32)
- new net ESPIO_33: J6.38 (Pin_38), U6.9 (IO33)
- new net ESPIO_34: J6.39 (Pin_39), U6.6 (IO34)
- new net ESPIO_35: J6.40 (Pin_40), U6.7 (IO35)
- new net ESPIO_36: J7.3 (Pin_3), U6.4 (SENSOR_VP)
- new net ESPIO_39: J7.2 (Pin_2), U6.5 (SENSOR_VN)
- new net ESPIO_4: J6.27 (Pin_27), U6.26 (IO4)
- new net ESPIO_5: J6.28 (Pin_28), U6.29 (IO5)
- new net ESP_D+: J2.A6 (D+), J2.B6 (D+), U5.3 (D+)
- new net ESP_D-: J2.A7 (D-), J2.B7 (D-), U5.4 (D-)
- new net GND: C1.2, C10.1, C11.1, C12.1, C13.2, C14.2, C15.2, C16.2, C17.2, C18.2, C19.2, C2.2, C20.2, C21.1, C22.2, C23.2, C24.2, C25.2, C26.1, C27.2, C28.2, C29.2, C3.2, C30.2, C31.2, C32.2, C4.2, C5.1, C6.1, C7.1, C8.1, C9.1, D4.1 (K), D5.1 (K), D7.1 (K), D8.2 (VSS), H1.1, H2.1, H3.1, H4.1, J1.A1 (GND), J1.A12 (GND), J1.B1 (GND), J1.B12 (GND), J1.SH (SHIELD), J2.A1 (GND), J2.A12 (GND), J2.B1 (GND), J2.B12 (GND), J2.SH (SHIELD), J3.6 (VSS), J3.SH (SHIELD), J4.2 (Pin_2), J5.3 (Pin_3), R1.2, R12.1, R2.2, R3.2, R4.2, R9.2, SW1.1, SW2.1, SW3.1, U1.19 (TESTEN), U1.57 (GND), U2.2 (GND), U3.2 (V_{SS}), U4.4 (GND), U5.2 (GND), U5.25 (GND), U6.[1,15,38,39] (GND), Y1.2
- new net QSPI_SCLK: U1.52 (QSPI_SCLK), U4.6 (CLK)
- new net QSPI_SD0: U1.53 (QSPI_SD0), U4.5 (DI/IO_{0})
- new net QSPI_SD1: U1.55 (QSPI_SD1), U4.2 (DO/IO_{1})
- new net QSPI_SD2: U1.54 (QSPI_SD2), U4.3 (~{WP}/IO_{2})
- new net QSPI_SD3: U1.51 (QSPI_SD3), U4.7 (~{HOLD}/~{RESET}/IO_{3})
- new net QSPI_SS: R15.2, R16.1, U1.56 (~{QSPI_SS}), U4.1 (~{CS})
- new net RPIO_0: J6.1 (Pin_1), U1.2 (GPIO0)
- new net RPIO_1: J6.2 (Pin_2), U1.3 (GPIO1)
- new net RPIO_12: J6.9 (Pin_9), U1.15 (GPIO12)
- new net RPIO_13: J6.10 (Pin_10), U1.16 (GPIO13)
- new net RPIO_14: J6.11 (Pin_11), U1.17 (GPIO14)
- new net RPIO_15: J6.12 (Pin_12), U1.18 (GPIO15)
- new net RPIO_16: J6.13 (Pin_13), U1.27 (GPIO16)
- new net RPIO_17: J6.14 (Pin_14), U1.28 (GPIO17)
- new net RPIO_18: J3.3 (CMD), J6.15 (Pin_15), U1.29 (GPIO18)
- new net RPIO_19: J3.7 (DAT0), J6.16 (Pin_16), U1.30 (GPIO19)
- new net RPIO_2: J6.3 (Pin_3), U1.4 (GPIO2)
- new net RPIO_20: J6.17 (Pin_17), U1.31 (GPIO20)
- new net RPIO_21: J6.18 (Pin_18), U1.32 (GPIO21)
- new net RPIO_22: J3.2 (DAT3/CD), J6.19 (Pin_19), U1.34 (GPIO22)
- new net RPIO_23: J6.20 (Pin_20), U1.35 (GPIO23)
- new net RPIO_24: J6.21 (Pin_21), U1.36 (GPIO24)
- new net RPIO_25: J6.22 (Pin_22), R14.1, U1.37 (GPIO25)
- new net RPIO_26: J6.23 (Pin_23), U1.38 (GPIO26/ADC0)
- new net RPIO_27: J6.24 (Pin_24), U1.39 (GPIO27/ADC1)
- new net RPIO_28: J6.25 (Pin_25), U1.40 (GPIO28/ADC2)
- new net RPIO_29: J6.26 (Pin_26), U1.41 (GPIO29/ADC3)
- new net RPIO_3: J6.4 (Pin_4), U1.5 (GPIO3)
- new net RPIO_4: J6.5 (Pin_5), U1.6 (GPIO4)
- new net RPIO_5: J3.5 (CLK), J6.6 (Pin_6), U1.7 (GPIO5)
- new net RPIO_6: J6.7 (Pin_7), U1.8 (GPIO6)
- new net RPIO_7: J6.8 (Pin_8), U1.9 (GPIO7)
- new net RPIO_RUN: J7.1 (Pin_1), U1.26 (RUN)
- new net RPUSB_D+: J1.A6 (D+), J1.B6 (D+), R8.2
- new net RPUSB_D-: J1.A7 (D-), J1.B7 (D-), R7.1
- new net RP_SWCLK: J8.3 (Pin_3), U1.24 (SWCLK)
- new net RP_SWDIO: J8.4 (Pin_4), U1.25 (SWDIO)
- new net RTS: R23.1, U5.19 (~{RTS})
- new net RXD0: U5.20 (RXD), U6.34 (RXD0/IO3)
- new net SD_DAT1: J3.8 (DAT1), R5.1
- new net SD_DAT2: J3.1 (DAT2), R6.1
- new net TXD0: U5.21 (TXD), U6.35 (TXD0/IO1)
- new net USB_BOOT: C22.1, R16.2, SW1.2
- new net VBAT: C18.1, J4.1 (Pin_1), Q1.3 (D), U3.3 (V_{BAT})
- new net VBUS: F1.2, J1.A4 (VBUS), J1.A9 (VBUS), J1.B4 (VBUS), J1.B9 (VBUS), J2.A4 (VBUS), J2.A9 (VBUS), J2.B4 (VBUS), J2.B9 (VBUS)
- new net XIN: C20.1, U1.20 (XIN), Y1.1
- new net XOUT: C21.2, R17.2, U1.21 (XOUT)
